File: source_kicad/aecp_Nano_V2.kicad_pcb (KiCad board)
At the start: 2 copper layers, 86.5 x 75 mm, 26 parts, among them P1 CONN_IGBT1, P10 FIX, P11 FIX, P12 CONN_SEL2, P13 CONN_DEP2, P14 MP3V5050, P2 CONN_IGBT2, P3 CONN_DEP, P4 CONN_SEL1, P5 CONN_12V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

Commit message: Add new schématic and new board under Kicad, also a new version under Arduino
Connections:
- U1 pad 10: Net-(P12-Pad1) -> Net-(U1-Pad10)
- U1 pad 7: Net-(U1-Pad7) -> Net-(P4-Pad1)
- U1 pad 8: Net-(P4-Pad1) -> Net-(U1-Pad8)
- U1 pad 9: Net-(U1-Pad9) -> Net-(P12-Pad1)
Routing:
- net Net-(P12-Pad1): track 13.8 -> 15.5 mm
- net Net-(P4-Pad1): track 9.06 -> 10.1 mm
