File: source_kicad/aecp_Nano_V2.sch (KiCad schematic (older format))
At the start: 25 parts, among them P1 CONN_IGBT1, P10 FIX, P11 FIX, P12 CONN_SEL2, P13 CONN_DEP2, P14 MP3V5050, P2 CONN_IGBT2, P3 CONN_DEP, P4 CONN_SEL1, P5 CONN_12V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

Commit message: Add new schématic and new board under Kicad, also a new version under Arduino
Connections:
- net at U1.10 (A6): no longer P12.1 (P1)
- net at U1.7 (A3): now also P4.1 (P1)
- net at U1.8 (A4(SDA)): no longer P4.1 (P1)
- net at U1.9 (A5(SCL)): now also P12.1 (P1)
Other:
- moved on the sheet: P12, P4
Changed lines of the file:
@@
 L CONN_01X02 P4
 U 1 1 570ABCA6
-P 5600 3000
-F 0 "P4" H 5677 3038 50  0000 L CNN
-F 1 "CONN_SEL1" H 5677 2947 50  0000 L CNN
-F 2 "Connect:bornier2" H 5600 3000 50  0001 C CNN
-F 3 "" H 5600 3000 50  0000 C CNN
-	1    5600 3000
-	1    0    0    -1
-$EndComp
-Wire Wire Line
-	5400 3050 5300 3050
+P 5600 2900
+F 0 "P4" H 5677 2938 50  0000 L CNN
+F 1 "CONN_SEL1" H 5677 2847 50  0000 L CNN
+F 2 "Connect:bornier2" H 5600 2900 50  0001 C CNN
+F 3 "" H 5600 2900 50  0000 C CNN
+	1    5600 2900
+	1    0    0    -1
+$EndComp
+Wire Wire Line
+	5400 2950 5300 2950
 Wire Wire Line
 	5300 2400 5300 4600
@@
 Wire Wire Line
 	5400 2400 5300 2400
-Connection ~ 5300 3050
+Connection ~ 5300 2950
 Wire Wire Line
 	5400 2300 5100 2300
@@
 NoConn ~ 3050 2500
 NoConn ~ 4450 2350
-NoConn ~ 4450 2850
-NoConn ~ 4450 3050
 NoConn ~ 4450 3250
 NoConn ~ 3050 3450
@@
 	2750 3150 3050 3150
 NoConn ~ 3050 2700
-Wire Wire Line
-	5400 2950 4450 2950
 NoConn ~ 4450 2750
 $Comp
@@
 L CONN_01X02 P12
 U 1 1 5765BC76
-P 5600 3250
-F 0 "P12" H 5677 3288 50  0000 L CNN
-F 1 "CONN_SEL2" H 5677 3197 50  0000 L CNN
-F 2 "Connect:bornier2" H 5600 3250 50  0001 C CNN
-F 3 "" H 5600 3250 50  0000 C CNN
-	1    5600 3250
-	1    0    0    -1
-$EndComp
-Wire Wire Line
-	5400 3200 4600 3200
-Wire Wire Line
-	4600 3200 4600 3150
-Wire Wire Line
-	4600 3150 4450 3150
-Wire Wire Line
-	5400 3300 5300 3300
-Connection ~ 5300 3300
+P 5600 3150
+F 0 "P12" H 5677 3188 50  0000 L CNN
+F 1 "CONN_SEL2" H 5677 3097 50  0000 L CNN
+F 2 "Connect:bornier2" H 5600 3150 50  0001 C CNN
+F 3 "" H 5600 3150 50  0000 C CNN
+	1    5600 3150
+	1    0    0    -1
+$EndComp
+Wire Wire Line
+	5400 3100 4600 3100
+Wire Wire Line
+	5400 3200 5300 3200
+Connection ~ 5300 3200
 $Comp
 L CONN_01X01 P1
@@
 	7000 3000 7700 3000
 Wire Wire Line
-	7700 3100 7000 3100
+	7000 3100 7700 3100
 $Comp
 L GND #PWR05
@@
 Connection ~ 7500 3100
 Connection ~ 7100 2900
+NoConn ~ 4450 3150
+Wire Wire Line
+	4600 3050 4450 3050
+NoConn ~ 4450 2950
+Wire Wire Line
+	4450 2850 5400 2850
+Wire Wire Line
+	4600 3100 4600 3050
 $EndSCHEMATC
