File: source_kicad/aecp_Nano_V3.kicad_pcb (KiCad board)
At the start: 2 copper layers, 86.5 x 88 mm, 27 parts, among them P1 CONN_IGBT, P10 FIX, P11 FIX, P12 CONN_SEL2, P13 CONN_DEP2, P14 MP3V5050, P3 CONN_DEP, P4 CONN_SEL1, P5 CONN_12V, P6 CONN_HALL1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

Commit message: New PCB version
Parts:
- removed the G1 at (82.4, 109.0)
- added P15: FIX, Connect:1pin, F.Cu at (135.0, 33.0)
- added P16: FIX, Connect:1pin, F.Cu at (142.0, 33.0)
- added P17: FIX, Connect:1pin, F.Cu at (135.0, 69.4)
- added P18: FIX, Connect:1pin, F.Cu at (142.0, 69.4)
- G2: value PanhardCD -> Panhard24CT
- moved P13 11.4 mm to (136.0, 37.8)
- moved P14 11.4 mm to (137.3, 55.4)
- moved C2 11.4 mm to (131.7, 42.8)
- moved C3 11.4 mm to (145.4, 42.8)
- moved G1 11.4 mm to (141.2, 55.4)
- moved G2 0.20 mm to (86.1, 71.4)
Other:
- outline, holes or cut-outs redrawn
- board text added: "SC"
- board text added: "SV"
- board text added: "Vac sensor"
- board text removed: "Dep sensor"
- board text removed: "S1"
- board text removed: "S2"
