File: source_kicad/aecp_Nano_V3.sch (KiCad schematic (older format))
At the start: 25 parts, among them P1 CONN_IGBT1, P10 FIX, P11 FIX, P12 CONN_SEL2, P13 CONN_DEP2, P14 MP3V5050, P2 CONN_IGBT2, P3 CONN_DEP, P4 CONN_SEL1, P5 CONN_12V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

Commit message: New version of the PCB
Parts:
- removed P1: CONN_IGBT1, Connect:1pin, symbol CONN_01X01
- removed P2: CONN_IGBT2, Connect:1pin, symbol CONN_01X01
- added G2: PanhardCD, aecp_Nano_V3:Panhard24CT3, symbol PanhardCD
- added P1: CONN_IGBT, Connect:bornier2, symbol CONN_01X02
Connections:
- net GND: now also P5.1 (P1); no longer P5.2 (P2)
- net at U3.1 (IN): now also P5.2 (P2); no longer P5.1 (P1)
- net at Q2.2 (C): now also P1.1 (P1)
- net at Q1.2 (C): now also P1.2 (P2)
Other:
- moved on the sheet: P6
Changed lines of the file:
@@
 LIBS:DDLM
 LIBS:Tete_budha
-LIBS:aecp_Nano_V2-cache
+LIBS:PanhardCD
+LIBS:aecp_Nano_V3-cache
 EELAYER 25 0
 EELAYER END
@@
 F 3 "" H 6450 1150 50  0000 C CNN
 	1    6450 1150
-	1    0    0    -1
+	1    0    0    1
 $EndComp
 $Comp
@@
 $EndComp
 Wire Wire Line
-	3050 3350 2000 3350
-Wire Wire Line
-	2100 3150 2000 3150
+	3050 3350 1950 3350
+Wire Wire Line
+	2100 3150 1950 3150
 Wire Wire Line
 	2100 1100 2100 3150
@@
 	2100 4600 2100 3250
 Wire Wire Line
-	2250 3250 2000 3250
+	2250 3250 1950 3250
 Connection ~ 3750 4600
 $Comp
@@
 	2350 1400 2350 1300
 Wire Wire Line
-	2350 1950 2350 1800
-Wire Wire Line
-	2400 1950 2350 1950
+	2350 1800 2350 2000
 Wire Wire Line
 	2350 2200 2350 2150
@@
 L CONN_01X03 P6
 U 1 1 570AD572
-P 1800 3250
-F 0 "P6" H 1719 2919 50  0000 C CNN
-F 1 "CONN_HALL1" H 1719 3010 50  0000 C CNN
-F 2 "Connect:bornier3" H 1800 3250 50  0001 C CNN
-F 3 "" H 1800 3250 50  0000 C CNN
-	1    1800 3250
+P 1750 3250
+F 0 "P6" H 1669 2919 50  0000 C CNN
+F 1 "CONN_HALL1" H 1669 3010 50  0000 C CNN
+F 2 "Connect:bornier3" H 1750 3250 50  0001 C CNN
+F 3 "" H 1750 3250 50  0000 C CNN
+	1    1750 3250
 	-1   0    0    1
 $EndComp
@@
 	5400 3200 5300 3200
 Connection ~ 5300 3200
-$Comp
-L CONN_01X01 P1
-U 1 1 5765C64A
-P 2600 1950
-F 0 "P1" H 2600 2050 50  0000 C CNN
-F 1 "CONN_IGBT1" V 2700 1950 50  0000 C CNN
-F 2 "Connect:1pin" H 2600 1950 50  0001 C CNN
-F 3 "" H 2600 1950 50  0000 C CNN
-	1    2600 1950
-	1    0    0    1
-$EndComp
-$Comp
-L CONN_01X01 P2
-U 1 1 5765C737
-P 2600 2750
-F 0 "P2" H 2600 2850 50  0000 C CNN
-F 1 "CONN_IGBT2" V 2700 2750 50  0000 C CNN
-F 2 "Connect:1pin" H 2600 2750 50  0001 C CNN
-F 3 "" H 2600 2750 50  0000 C CNN
-	1    2600 2750
-	1    0    0    -1
-$EndComp
-Wire Wire Line
-	2350 2750 2400 2750
 Wire Wire Line
 	2350 2150 2250 2150
@@
 Wire Wire Line
 	4600 3100 4600 3050
+$Comp
+L PanhardCD G2
+U 1 1 5801C6F1
+P 7750 4150
+F 0 "G2" H 7750 3792 60  0001 C CNN
+F 1 "PanhardCD" H 7750 4508 60  0001 C CNN
+F 2 "aecp_Nano_V3:Panhard24CT3" H 7750 4150 60  0001 C CNN
+F 3 "" H 7750 4150 60  0001 C CNN
+	1    7750 4150
+	1    0    0    -1
+$EndComp
+$Comp
+L CONN_01X02 P1
+U 1 1 58026BF1
+P 1750 2050
+F 0 "P1" H 1827 2088 50  0000 L CNN
+F 1 "CONN_IGBT" H 1827 1997 50  0000 L CNN
+F 2 "Connect:bornier2" H 1750 2050 50  0001 C CNN
+F 3 "" H 1750 2050 50  0000 C CNN
+	1    1750 2050
+	-1   0    0    1
+$EndComp
+Wire Wire Line
+	2000 2100 2000 2750
+Wire Wire Line
+	2000 2750 2350 2750
+Wire Wire Line
+	2350 2000 1950 2000
+Wire Wire Line
+	2000 2100 1950 2100
 $EndSCHEMATC

Commit message: New PCB version
Parts:
- removed G2: PanhardCD, aecp_Nano_V3:Panhard24CT3, symbol PanhardCD
- added G2: 24CT, DDLM:Panhard24CT, symbol 24CT
- added P15, P16, P17, P18: FIX, Mounting_Holes:MountingHole_2.2mm_M2_Pad_Via, symbol TST
Changed lines of the file:
@@
 LIBS:DDLM
 LIBS:Tete_budha
-LIBS:PanhardCD
+LIBS:Panhard
 LIBS:aecp_Nano_V3-cache
 EELAYER 25 0
@@
 	4600 3100 4600 3050
 $Comp
-L PanhardCD G2
-U 1 1 5801C6F1
-P 7750 4150
-F 0 "G2" H 7750 3792 60  0001 C CNN
-F 1 "PanhardCD" H 7750 4508 60  0001 C CNN
-F 2 "aecp_Nano_V3:Panhard24CT3" H 7750 4150 60  0001 C CNN
-F 3 "" H 7750 4150 60  0001 C CNN
-	1    7750 4150
-	1    0    0    -1
-$EndComp
-$Comp
 L CONN_01X02 P1
 U 1 1 58026BF1
@@
 Wire Wire Line
 	2000 2100 1950 2100
+$Comp
+L TST P18
+U 1 1 5807D293
+P 9100 1800
+F 0 "P18" H 9178 1940 50  0000 L CNN
+F 1 "FIX" H 9178 1849 50  0000 L CNN
+F 2 "Mounting_Holes:MountingHole_2.2mm_M2_Pad_Via" H 9100 1800 50  0001 C CNN
+F 3 "" H 9100 1800 50  0000 C CNN
+	1    9100 1800
+	1    0    0    -1
+$EndComp
+$Comp
+L TST P15
+U 1 1 5807D31D
+P 8350 1800
+F 0 "P15" H 8428 1940 50  0000 L CNN
+F 1 "FIX" H 8428 1849 50  0000 L CNN
+F 2 "Mounting_Holes:MountingHole_2.2mm_M2_Pad_Via" H 8350 1800 50  0001 C CNN
+F 3 "" H 8350 1800 50  0000 C CNN
+	1    8350 1800
+	1    0    0    -1
+$EndComp
+$Comp
+L TST P16
+U 1 1 5807D404
+P 8600 1800
+F 0 "P16" H 8678 1940 50  0000 L CNN
+F 1 "FIX" H 8678 1849 50  0000 L CNN
+F 2 "Mounting_Holes:MountingHole_2.2mm_M2_Pad_Via" H 8600 1800 50  0001 C CNN
+F 3 "" H 8600 1800 50  0000 C CNN
+	1    8600 1800
+	1    0    0    -1
+$EndComp
+$Comp
+L TST P17
+U 1 1 5807D40A
+P 8850 1800
+F 0 "P17" H 8928 1940 50  0000 L CNN
+F 1 "FIX" H 8928 1849 50  0000 L CNN
+F 2 "Mounting_Holes:MountingHole_2.2mm_M2_Pad_Via" H 8850 1800 50  0001 C CNN
+F 3 "" H 8850 1800 50  0000 C CNN
+	1    8850 1800
+	1    0    0    -1
+$EndComp
+$Comp
+L 24CT G2
+U 1 1 580BB541
+P 7850 4450
+F 0 "G2" H 7850 3527 60  0001 C CNN
+F 1 "24CT" H 7850 5373 60  0001 C CNN
+F 2 "DDLM:Panhard24CT" H 7850 4450 60  0001 C CNN
+F 3 "" H 7850 4450 60  0001 C CNN
+	1    7850 4450
+	1    0    0    -1
+$EndComp
 $EndSCHEMATC
