File: source_kicad/aecp_Nano_V3_main_board.kicad_pcb (KiCad board)
At the start: 2 copper layers, 86.5 x 88 mm, 30 parts, among them P1 CONN_IGBT, P10 FIX, P11 FIX, P12 CONN_SEL2, P13 CONN_DEP2, P14 MP3V5050, P15 FIX, P16 FIX, P17 FIX, P18 FIX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

Commit message: Last version of PCB with gerber files
Parts:
- removed C2: 1µ, Capacitors_ThroughHole:C_Rect_L7_W3.5_P5
- removed C3: 470p, Capacitors_ThroughHole:C_Rect_L7_W3.5_P5
- removed the G1 at (142.4, 55.3)
- removed P13: CONN_DEP2, Socket_Strips:Socket_Strip_Straight_1x03
- removed P14: MP3V5050, MP3V5050V:MP3V5050V
- removed P15, P16, P17, P18: FIX, Connect:1pin
- removed P7: CONN_HALL2, Socket_Strips:Socket_Strip_Straight_1x03
- removed U2: A3144, TO_SOT_Packages_THT:TO-92_Horizontal2_Inline_Narrow_Oval
Routing:
- net GND: track 202.0 -> 161.7 mm
- net Net-(P7-Pad3): track 13.2 -> 0.00 mm
- net Net-(P7-Pad1): track 13.2 -> 0.00 mm
- net Net-(C2-Pad2): track 13.1 -> 0.00 mm
- net Net-(C3-Pad2): track 13.1 -> 0.00 mm
- net Net-(P7-Pad2): track 12.9 -> 0.00 mm
Other:
- board size 86.5 x 88 mm -> 49.5 x 88 mm
- board text removed: "A3144"
- board text removed: "G"
- board text removed: "O"
- board text removed: "Out"
- board text removed: "V"
- board text removed: "Vcc"

Commit message: Bug corrected in the PCB
Parts:
- G2: value Panhard24CT -> 24CT
Connections:
- U1 pad 7: Net-(P4-Pad1) -> Net-(U1-Pad7)
- U1 pad 8: Net-(U1-Pad8) -> Net-(P4-Pad1)
Routing:
- net Net-(P4-Pad1): track 12.2 -> 9.98 mm
Changed lines of the file:
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@@
     (links 23)
     (no_connects 1)
-    (area 61.249999 27.249999 124.182 121.556881)
+    (area 61.249999 27.249999 163.781212 121.556881)
     (thickness 1.6)
     (drawings 33)
-    (tracks 106)
+    (tracks 104)
     (zones 0)
     (modules 19)
@@
       (layerselection 0x010f0_80000001)
       (usegerberextensions false)
-      (excludeedgelayer true)
+      (excludeedgelayer false)
       (linewidth 0.100000)
       (plotframeref false)
@@
       (padsonsilk false)
       (subtractmaskfromsilk false)
-      (outputformat 1)
+      (outputformat 2)
       (mirror false)
-      (drillshape 0)
+      (drillshape 2)
       (scaleselection 1)
-      (outputdirectory "gerber/aecp main board/"))
+      (outputdirectory ""))
   )
   (net 0 "")
@@
   (net 31 "Net-(U1-Pad6)")
   (net 32 "Net-(P12-Pad1)")
-  (net 33 "Net-(U1-Pad8)")
-  (net 34 "Net-(U1-Pad10)")
-  (net 35 "Net-(P1-Pad2)")
-  (net 36 "Net-(P5-Pad2)")
+  (net 33 "Net-(U1-Pad10)")
+  (net 34 "Net-(P1-Pad2)")
+  (net 35 "Net-(P5-Pad2)")
+  (net 36 "Net-(U1-Pad7)")
   (net_class Default "Ceci est la Netclass par défaut"
     (clearance 0.2)
@@
     (add_net "Net-(U1-Pad5)")
     (add_net "Net-(U1-Pad6)")
-    (add_net "Net-(U1-Pad8)")
+    (add_net "Net-(U1-Pad7)")
   )
   (module Connect:bornier2 (layer F.Cu)
@@
       (net 31 "Net-(U1-Pad6)"))
     (pad 7 thru_hole oval (at -3.81 7.62 270) (size 1.5748 2.286) (drill 1.016) (layers *.Cu *.Mask F.SilkS)
-      (net 20 "Net-(P4-Pad1)"))
+      (net 36 "Net-(U1-Pad7)"))
     (pad 8 thru_hole oval (at -1.27 7.62 270) (size 1.5748 2.286) (drill 1.016) (layers *.Cu *.Mask F.SilkS)
-      (net 33 "Net-(U1-Pad8)"))
+      (net 20 "Net-(P4-Pad1)"))
     (pad 9 thru_hole oval (at 1.27 7.62 270) (size 1.5748 2.286) (drill 1.016) (layers *.Cu *.Mask F.SilkS)
       (net 32 "Net-(P12-Pad1)"))
     (pad 10 thru_hole oval (at 3.81 7.62 270) (size 1.5748 2.286) (drill 1.016) (layers *.Cu *.Mask F.SilkS)
-      (net 34 "Net-(U1-Pad10)"))
+      (net 33 "Net-(U1-Pad10)"))
     (pad 11 thru_hole oval (at 6.35 7.62 270) (size 1.5748 2.286) (drill 1.016) (layers *.Cu *.Mask F.SilkS)
       (net 3 "Net-(U1-Pad11)"))
@@
       (net 9 GND))
     (pad 2 thru_hole circle (at 2.54 0 270) (size 2.54 2.54) (drill 1.524) (layers *.Cu *.Mask F.SilkS)
-      (net 36 "Net-(P5-Pad2)"))
+      (net 35 "Net-(P5-Pad2)"))
     (model walter/conn_screw/mors_2p.wrl
       (at (xyz 0 0 0))
@@
     (fp_line (start 0 -3.048) (end 5.334 -3.048) (layer F.SilkS) (width 0.15))
     (pad 2 thru_hole oval (at 0 0) (size 2.49936 1.50114) (drill 1.016) (layers *.Cu *.Mask F.SilkS)
-      (net 35 "Net-(P1-Pad2)"))
+      (net 34 "Net-(P1-Pad2)"))
     (pad 1 thru_hole oval (at -2.54 0) (size 2.49936 1.50114) (drill 1.016) (layers *.Cu *.Mask F.SilkS)
       (net 23 "Net-(Q1-Pad1)"))
@@
       (net 9 GND))
     (pad 1 thru_hole oval (at -2.54 0 90) (size 3.50012 1.69926) (drill 1.016) (layers *.Cu *.Mask F.SilkS)
-      (net 36 "Net-(P5-Pad2)"))
+      (net 35 "Net-(P5-Pad2)"))
     (pad 3 thru_hole oval (at 2.54 0 90) (size 3.50012 1.69926) (drill 1.016) (layers *.Cu *.Mask F.SilkS)
       (net 22 +5V))
@@
       (net 17 "Net-(P1-Pad1)"))
     (pad 2 thru_hole circle (at 2.54 0 270) (size 2.54 2.54) (drill 1.524) (layers *.Cu *.Mask F.SilkS)
-      (net 35 "Net-(P1-Pad2)"))
+      (net 34 "Net-(P1-Pad2)"))
     (model walter/conn_screw/mors_2p.wrl
       (at (xyz 0 0 0))
@@
       (effects (font (thickness 0.3)) (justify mirror))
     )
-    (fp_text value Panhard24CT (at 0.75 0 270) (layer B.SilkS) hide
+    (fp_text value 24CT (at 0.75 0 270) (layer B.SilkS) hide
       (effects (font (thickness 0.3)) (justify mirror))
     )
@@
   (segment (start 75.57008 53.9623) (end 70.78218 58.7502) (width 2.032) (layer B.Cu) (net 19))
   (segment (start 77.29982 53.98516) (end 77.32268 53.9623) (width 1.016) (layer B.Cu) (net 19) (status 30))
+  (segment (start 77.32268 64.1223) (end 74.40168 64.1223) (width 1.524) (layer B.Cu) (net 20))
+  (segment (start 74.40168 64.1223) (end 69.46138 69.0626) (width 1.524) (layer B.Cu) (net 20))
   (segment (start 69.46138 69.0626) (end 69.53758 69.0626) (width 1.524) (layer B.Cu) (net 20))
-  (segment (start 69.53758 69.0626) (end 73.41108 65.1891) (width 1.524) (layer B.Cu) (net 20))
-  (segment (start 73.41108 65.1891) (end 73.41108 63.1317) (width 1.524) (layer B.Cu) (net 20))
-  (segment (start 73.41108 63.1317) (end 74.96048 61.5823) (width 1.524) (layer B.Cu) (net 20))
-  (segment (start 74.96048 61.5823) (end 77.32268 61.5823) (width 1.524) (layer B.Cu) (net 20))
   (segment (start 69.48678 38.227) (end 81.62798 38.227) (width 2.032) (layer B.Cu) (net 21))
   (segment (start 89.98458 71.7423) (end 92.56268 71.7423) (width 2.032) (layer B.Cu) (net 21))
@@
   (segment (start 71.44258 79.3877) (end 69.43598 79.3877) (width 1.524) (layer B.Cu) (net 32))
   (via (at 69.43598 79.3877) (size 0.6) (drill 0.4) (layers F.Cu B.Cu) (net 32))
-  (segment (start 98.45548 53.58384) (end 102.91572 53.58384) (width 2.032) (layer B.Cu) (net 35))
-  (segment (start 75.29576 105.1052) (end 69.41058 105.1052) (width 2.032) (layer B.Cu) (net 35))
-  (segment (start 78.74 108.54944) (end 75.29576 105.1052) (width 2.032) (layer B.Cu) (net 35))
-  (segment (start 104.06888 108.54944) (end 78.74 108.54944) (width 2.032) (layer B.Cu) (net 35))
-  (segment (start 107.62996 104.98836) (end 104.06888 108.54944) (width 2.032) (layer B.Cu) (net 35))
-  (segment (start 107.62996 58.29808) (end 107.62996 104.98836) (width 2.032) (layer B.Cu) (net 35))
-  (segment (start 102.91572 53.58384) (end 107.62996 58.29808) (width 2.032) (layer B.Cu) (net 35))
-  (segment (start 69.42328 94.7674) (end 78.82128 94.7674) (width 2.032) (layer B.Cu) (net 36))
-  (segment (start 78.82128 94.7674) (end 82.40268 98.3488) (width 2.032) (layer B.Cu) (net 36))
-  (segment (start 82.37728 98.3234) (end 82.40268 98.3488) (width 1.524) (layer B.Cu) (net 36) (status 30))
+  (segment (start 98.45548 53.58384) (end 102.91572 53.58384) (width 2.032) (layer B.Cu) (net 34))
+  (segment (start 75.29576 105.1052) (end 69.41058 105.1052) (width 2.032) (layer B.Cu) (net 34))
+  (segment (start 78.74 108.54944) (end 75.29576 105.1052) (width 2.032) (layer B.Cu) (net 34))
+  (segment (start 104.06888 108.54944) (end 78.74 108.54944) (width 2.032) (layer B.Cu) (net 34))
+  (segment (start 107.62996 104.98836) (end 104.06888 108.54944) (width 2.032) (layer B.Cu) (net 34))
+  (segment (start 107.62996 58.29808) (end 107.62996 104.98836) (width 2.032) (layer B.Cu) (net 34))
+  (segment (start 102.91572 53.58384) (end 107.62996 58.29808) (width 2.032) (layer B.Cu) (net 34))
+  (segment (start 69.42328 94.7674) (end 78.82128 94.7674) (width 2.032) (layer B.Cu) (net 35))
+  (segment (start 78.82128 94.7674) (end 82.40268 98.3488) (width 2.032) (layer B.Cu) (net 35))
+  (segment (start 82.37728 98.3234) (end 82.40268 98.3488) (width 1.524) (layer B.Cu) (net 35) (status 30))
 )
